Commit message: added custom models

File: src/gazebo/kinova_description/urdf/j2n6s300_standalone.xacro (robot description, xacro)
@@ -21,5 +21,5 @@
     <child link="root" />
     <parent link="world" />
-    <origin xyz="0 0 0" rpy="0 0 0" />
+    <origin xyz="0 0 1.0" rpy="0 0 0" />
   </joint>
   <xacro:property name="robot_root" value="root" />
